Commit message: Add PID parameter to wheel joint for gazebo ros2 control

File: urdf/ros2_control.hsrc1s.gazebo.xacro (robot description, xacro)
@@ -58,5 +58,5 @@
          <plugin>gazebo_ros2_control/GazeboSystem</plugin>
       </hardware>
-      <xacro:macro name="gazebo_velocity_joint" params="name">
+      <xacro:macro name="gazebo_velocity_joint" params="name p_gain i_gain d_gain">
         <joint name="${name}">
           <command_interface name="velocity" />
@@ -64,4 +64,8 @@
           <state_interface name="velocity" />
           <state_interface name="effort" />
+          <param name="p_gain">${p_gain}</param>
+          <param name="i_gain">${i_gain}</param>
+          <param name="d_gain">${d_gain}</param>
+          <param name="i_max">3.0</param>
         </joint>
       </xacro:macro>
@@ -93,6 +97,6 @@
       <xacro:gazebo_position_joint name="wrist_roll_joint" p_gain="900.0" i_gain="0.0" d_gain="0.0"/>
       <xacro:gazebo_position_joint name="base_roll_joint" p_gain="900.0" i_gain="200.0" d_gain="100.0"/>
-      <xacro:gazebo_velocity_joint name="base_r_drive_wheel_joint" />
-      <xacro:gazebo_velocity_joint name="base_l_drive_wheel_joint" />
+      <xacro:gazebo_velocity_joint name="base_r_drive_wheel_joint" p_gain="35.0" i_gain="0.5" d_gain="0.0"/>
+      <xacro:gazebo_velocity_joint name="base_l_drive_wheel_joint" p_gain="35.0" i_gain="0.5" d_gain="0.0"/>
       <xacro:gazebo_read_only_joint name="hand_motor_joint" />
       <xacro:gazebo_read_only_joint name="hand_l_spring_proximal_joint" />
