Commit message: Update robot model parameters

File: urdf/base_v2/base.gazebo.xacro (robot description, xacro)
@@ -26,4 +26,6 @@
 -->
 <robot xmlns:xacro="http://ros.org/wiki/xacro">
+    <xacro:arg name="ground_truth_xyz_offset" default="0.0\ 0.0\ 0.0"/>
+    <xacro:arg name="ground_truth_rpy_offset" default="0.0\ 0.0\ 0.0"/>
     <xacro:macro name="hsrb_base_gazebo" params="prefix robot_namespace">
         <xacro:gazebo_link name="${prefix}_link" gravity="true" collide="false" friction="0.9"/>
@@ -37,4 +39,17 @@
         <xacro:gazebo_link_bumper name="${prefix}_f_bumper" robot_namespace="${robot_namespace}" gravity="true" collide="false" friction="0.9"/>
         <xacro:gazebo_link_bumper name="${prefix}_b_bumper" robot_namespace="${robot_namespace}" gravity="true" collide="false" friction="0.9"/>
+        <gazebo>
+            <plugin name="odom_ground_truth" filename="libtmc_gazebo_ros_p3d.so">
+                <body_name>${prefix}_footprint</body_name>
+                <frame_name>map</frame_name>
+                <update_rate>30</update_rate>
+                <xyz_offset>$(arg ground_truth_xyz_offset)</xyz_offset>
+                <rpy_offset>$(arg ground_truth_rpy_offset)</rpy_offset>
+                <ros>
+                    <namespace>${robot_namespace}</namespace>
+                    <remapping>odom:=odom_ground_truth</remapping>
+                </ros>
+            </plugin>
+        </gazebo>
     </xacro:macro>
 </robot>

File: urdf/base_v2/base.urdf.xacro (robot description, xacro)
@@ -37,5 +37,5 @@
     <xacro:property name="passive_wheel_offset_x" value="0.1495" />
     <xacro:property name="passive_wheel_offset_y" value="0.055" />
-    <xacro:property name="drive_wheel_max_effort" value="11.067" />
+    <xacro:property name="drive_wheel_max_effort" value="28.0" />
     <xacro:property name="drive_wheel_max_velocity" value="20.8" />
     <xacro:property name="roll_joint_max_effort" value="34.46" />

File: urdf/base_v3/base.urdf.xacro (robot description, xacro)
@@ -37,5 +37,5 @@
     <xacro:property name="passive_wheel_offset_x" value="0.1665" />
     <xacro:property name="passive_wheel_offset_y" value="0.055" />
-    <xacro:property name="drive_wheel_max_effort" value="11.067" />
+    <xacro:property name="drive_wheel_max_effort" value="28.0" />
     <xacro:property name="drive_wheel_max_velocity" value="20.8" />
     <xacro:property name="roll_joint_max_effort" value="34.46" />

File: urdf/ros2_control.hsrb4s.gazebo.xacro (robot description, xacro)
@@ -54,4 +54,17 @@
         </parameters>
       </plugin>
+      <plugin name="grasp_hack_plugin" filename="libtmc_gazebo_grasp_hack_hrh_gripper.so">
+        <grasp_check>
+          <attach_steps>1</attach_steps>
+          <detach_steps>2</detach_steps>
+          <min_contact_count>1</min_contact_count>
+          <max_attach_weight>1.2</max_attach_weight>
+        </grasp_check>
+        <gripper_link>hand_r_distal_link</gripper_link>
+        <gripper_link>hand_l_distal_link</gripper_link>
+        <gripper_link>hand_r_spring_proximal_link</gripper_link>
+        <gripper_link>hand_l_spring_proximal_link</gripper_link>
+        <palm_link>wrist_ft_sensor_frame</palm_link>
+      </plugin>
     </gazebo>
     <ros2_control name="GazeboSystem" type="system">
@@ -93,9 +106,9 @@
       <xacro:gazebo_position_joint name="head_pan_joint" p_gain="1200.0" i_gain="0.0" d_gain="10.0"/>
       <xacro:gazebo_position_joint name="arm_lift_joint" p_gain="900.0" i_gain="200.0" d_gain="100.0"/>
-      <xacro:gazebo_position_joint name="arm_flex_joint" p_gain="2000.0" i_gain="10.0" d_gain="20.0"/>
+      <xacro:gazebo_position_joint name="arm_flex_joint" p_gain="2000.0" i_gain="100.0" d_gain="20.0"/>
       <xacro:gazebo_position_joint name="arm_roll_joint" p_gain="1000.0" i_gain="10.0" d_gain="1.0"/>
       <xacro:gazebo_position_joint name="wrist_flex_joint" p_gain="900.0" i_gain="1.0" d_gain="30.0"/>
       <xacro:gazebo_position_joint name="wrist_roll_joint" p_gain="900.0" i_gain="1.0" d_gain="10.0"/>
-      <xacro:gazebo_position_joint name="base_roll_joint" p_gain="900.0" i_gain="200.0" d_gain="100.0"/>
+      <xacro:gazebo_position_joint name="base_roll_joint" p_gain="1000.0" i_gain="1.0" d_gain="10.0"/>
       <xacro:gazebo_velocity_joint name="base_r_drive_wheel_joint" p_gain="35.0" i_gain="0.5" d_gain="0.0"/>
       <xacro:gazebo_velocity_joint name="base_l_drive_wheel_joint" p_gain="35.0" i_gain="0.5" d_gain="0.0"/>

File: urdf/ros2_control.hsrb4s.robot.xacro (robot description, xacro)
@@ -34,10 +34,10 @@
         <joint name="${name}">
           <command_interface name="position">
-            <param name="min">"${min_angle}"</param>
-            <param name="max">"${max_angle}"</param>
+            <param name="min">${min_angle}</param>
+            <param name="max">${max_angle}</param>
           </command_interface>
           <command_interface name="velocity">
-            <param name="min">>${-velocity_limit}</param>
-            <param name="max">>${velocity_limit}</param>
+            <param name="min">${-velocity_limit}</param>
+            <param name="max">${velocity_limit}</param>
           </command_interface>
           <state_interface name="position"/>
@@ -56,6 +56,6 @@
         <joint name="${name}">
           <command_interface name="position">
-            <param name="min">"${min_angle}"</param>
-            <param name="max">"${max_angle}"</param>
+            <param name="min">${min_angle}</param>
+            <param name="max">${max_angle}</param>
           </command_interface>
           <state_interface name="position"/>
@@ -79,5 +79,5 @@
                         reduction="40.273862263"
                         drive_mode="5"
-                        velocity_limit="1.0"
+                        velocity_limit="6.05"
                         gear_ratio="0.002407705"
                         torque_constant="0.0174"/>
@@ -142,5 +142,5 @@
                                   reduction="1.0"
                                   drive_mode="0"
-                                  velocity_limit="1.0"
+                                  velocity_limit="3.0"
                                   gear_ratio="0.005090909"
                                   torque_constant="0.0184"

File: urdf/ros2_control.hsrc1s.gazebo.xacro (robot description, xacro)
@@ -53,4 +53,17 @@
         </parameters>
       </plugin>
+      <plugin name="grasp_hack_plugin" filename="libtmc_gazebo_grasp_hack_hrh_gripper.so">
+        <grasp_check>
+          <attach_steps>1</attach_steps>
+          <detach_steps>2</detach_steps>
+          <min_contact_count>1</min_contact_count>
+          <max_attach_weight>1.2</max_attach_weight>
+        </grasp_check>
+        <gripper_link>hand_r_distal_link</gripper_link>
+        <gripper_link>hand_l_distal_link</gripper_link>
+        <gripper_link>hand_r_spring_proximal_link</gripper_link>
+        <gripper_link>hand_l_spring_proximal_link</gripper_link>
+        <palm_link>wrist_ft_sensor_frame</palm_link>
+      </plugin>
     </gazebo>
     <ros2_control name="GazeboSystem" type="system">
@@ -58,4 +71,16 @@
          <plugin>gazebo_ros2_control/GazeboSystem</plugin>
       </hardware>
+      <xacro:macro name="gazebo_position_joint" params="name p_gain i_gain d_gain">
+        <joint name="${name}">
+          <command_interface name="position" />
+          <state_interface name="position" />
+          <state_interface name="velocity" />
+          <state_interface name="effort" />
+          <param name="p_gain">${p_gain}</param>
+          <param name="i_gain">${i_gain}</param>
+          <param name="d_gain">${d_gain}</param>
+          <param name="i_max">200.0</param>
+        </joint>
+      </xacro:macro>
       <xacro:macro name="gazebo_velocity_joint" params="name p_gain i_gain d_gain">
         <joint name="${name}">
@@ -70,16 +95,4 @@
         </joint>
       </xacro:macro>
-      <xacro:macro name="gazebo_position_joint" params="name p_gain i_gain d_gain">
-        <joint name="${name}">
-          <command_interface name="position" />
-          <state_interface name="position" />
-          <state_interface name="velocity" />
-          <state_interface name="effort" />
-          <param name="p_gain">${p_gain}</param>
-          <param name="i_gain">${i_gain}</param>
-          <param name="d_gain">${d_gain}</param>
-          <param name="i_max">200.0</param>
-        </joint>
-      </xacro:macro>
       <xacro:macro name="gazebo_read_only_joint" params="name">
         <joint name="${name}">
@@ -92,9 +105,9 @@
       <xacro:gazebo_position_joint name="head_pan_joint" p_gain="1200.0" i_gain="0.0" d_gain="10.0"/>
       <xacro:gazebo_position_joint name="arm_lift_joint" p_gain="900.0" i_gain="200.0" d_gain="100.0"/>
-      <xacro:gazebo_position_joint name="arm_flex_joint" p_gain="2000.0" i_gain="10.0" d_gain="20.0"/>
+      <xacro:gazebo_position_joint name="arm_flex_joint" p_gain="2000.0" i_gain="100.0" d_gain="20.0"/>
       <xacro:gazebo_position_joint name="arm_roll_joint" p_gain="1000.0" i_gain="10.0" d_gain="1.0"/>
       <xacro:gazebo_position_joint name="wrist_flex_joint" p_gain="900.0" i_gain="0.0" d_gain="0.0"/>
       <xacro:gazebo_position_joint name="wrist_roll_joint" p_gain="900.0" i_gain="0.0" d_gain="0.0"/>
-      <xacro:gazebo_position_joint name="base_roll_joint" p_gain="900.0" i_gain="200.0" d_gain="100.0"/>
+      <xacro:gazebo_position_joint name="base_roll_joint" p_gain="1000.0" i_gain="1.0" d_gain="10.0"/>
       <xacro:gazebo_velocity_joint name="base_r_drive_wheel_joint" p_gain="35.0" i_gain="0.5" d_gain="0.0"/>
       <xacro:gazebo_velocity_joint name="base_l_drive_wheel_joint" p_gain="35.0" i_gain="0.5" d_gain="0.0"/>

File: urdf/ros2_control.hsrc1s.robot.xacro (robot description, xacro)
@@ -34,10 +34,10 @@
         <joint name="${name}">
           <command_interface name="position">
-            <param name="min">"${min_angle}"</param>
-            <param name="max">"${max_angle}"</param>
+            <param name="min">${min_angle}</param>
+            <param name="max">${max_angle}</param>
           </command_interface>
           <command_interface name="velocity">
-            <param name="min">>${-velocity_limit}</param>
-            <param name="max">>${velocity_limit}</param>
+            <param name="min">${-velocity_limit}</param>
+            <param name="max">${velocity_limit}</param>
           </command_interface>
           <state_interface name="position"/>
@@ -56,6 +56,6 @@
         <joint name="${name}">
           <command_interface name="position">
-            <param name="min">"${min_angle}"</param>
-            <param name="max">"${max_angle}"</param>
+            <param name="min">${min_angle}</param>
+            <param name="max">${max_angle}</param>
           </command_interface>
           <state_interface name="position"/>
@@ -79,5 +79,5 @@
                         reduction="40.273862263"
                         drive_mode="5"
-                        velocity_limit="6.28"
+                        velocity_limit="6.05"
                         gear_ratio="0.002407705"
                         torque_constant="0.0174"/>
@@ -142,5 +142,5 @@
                                   reduction="1.0"
                                   drive_mode="0"
-                                  velocity_limit="1.0"
+                                  velocity_limit="3.0"
                                   gear_ratio="0.005090909"
                                   torque_constant="0.0184"

File: urdf/ros2_control.rviz.xacro (robot description, xacro)
@@ -32,4 +32,5 @@
         <param name="fake_sensor_commands">False</param>
         <param name="state_following_offset">0.0</param>
+        <param name="calculate_dynamics">True</param>
       </hardware>
       <xacro:macro name="rviz_joint" params="name">

File: urdf/sensors/hokuyo_laser.gazebo.xacro (robot description, xacro)
@@ -23,9 +23,8 @@
                     </range>
                 </ray>
-                <plugin name="hokuyo_laser" filename="libgazebo_ros_ray_sensor.so">
+                <plugin name="${sensor_name}" filename="libgazebo_ros_ray_sensor.so">
                     <output_type>sensor_msgs/LaserScan</output_type>
                     <frame_name>${frame_name}</frame_name>
                     <ros>
-                        <namespace>${robot_namespace}</namespace>
                         <remapping>~/out:=${ros_topic}</remapping>
                     </ros>

File: urdf/sensors/hokuyo_laser.urdf.xacro (robot description, xacro)
@@ -3,5 +3,5 @@
     <xacro:include filename="$(find hsrb_description)/urdf/sensors/hokuyo_laser.gazebo.xacro"/>
     <!-- range sensor -->
-    <xacro:macro name="hokuyo_laser" params="prefix robot_namespace parent min_angle max_angle *origin">
+    <xacro:macro name="hokuyo_laser" params="prefix robot_namespace parent min_angle max_angle ros_topic:='scan' *origin">
         <joint name="${prefix}_range_sensor_joint" type="fixed">
             <xacro:insert_block name="origin" />
@@ -29,5 +29,5 @@
             sensor_name="${prefix}_range_sensor"
             robot_namespace="${robot_namespace}"
-            ros_topic="scan"
+            ros_topic="${ros_topic}"
             frame_name="${prefix}_range_sensor_link"
             min_angle="${min_angle}" max_angle="${max_angle}" />
