Commit message: fixed description

File: robots/hsrb4s.urdf.xacro (robot description, xacro)
@@ -37,5 +37,5 @@
     <xacro:include filename="$(find hsrb_description)/urdf/hand_v0/hand.urdf.xacro" />
     <xacro:arg name="gazebo_sim" default="False"/>
-    <xacro:arg name="rviz_sim" default="False"/>
+    <xacro:arg name="rviz_sim" default="True"/>
     <xacro:arg name="personal_name" default=""/>
     <xacro:arg name="ground_truth_xyz_offset" default="0.0\ 0.0\ 0.0"/>
@@ -72,5 +72,5 @@
     <xacro:if value="$(arg rviz_sim)">
       <xacro:include filename="$(find hsrb_description)/urdf/ros2_control.rviz.xacro" />
-      <xacro:ros2_contorl_rviz/>
+      <xacro:ros2_control_rviz/>
     </xacro:if>
 </robot>

File: urdf/arm_v0/arm.urdf.xacro (robot description, xacro)
@@ -46,10 +46,10 @@
             <visual>
                 <geometry>
-                    <mesh filename="package://hsrb_meshes/meshes/arm_v0/shoulder.dae" />
+                    <mesh filename="package://hsrb_description/meshes/arm_v0/shoulder.dae" />
                 </geometry>
             </visual>
             <collision>
                 <geometry>
-                    <mesh filename="package://hsrb_meshes/meshes/arm_v0/shoulder.stl" />
+                    <mesh filename="package://hsrb_description/meshes/arm_v0/shoulder.stl" />
                 </geometry>
             </collision>
@@ -72,10 +72,10 @@
             <visual>
                 <geometry>
-                    <mesh filename="package://hsrb_meshes/meshes/arm_v0/arm_flex_light.dae" />
+                    <mesh filename="package://hsrb_description/meshes/arm_v0/arm_flex_light.dae" />
                 </geometry>
             </visual>
             <collision>
                 <geometry>
-                    <mesh filename="package://hsrb_meshes/meshes/arm_v0/arm_flex.stl" />
+                    <mesh filename="package://hsrb_description/meshes/arm_v0/arm_flex.stl" />
                 </geometry>
             </collision>
@@ -98,10 +98,10 @@
             <visual>
                 <geometry>
-                    <mesh filename="package://hsrb_meshes/meshes/arm_v0/arm_roll_light.dae" />
+                    <mesh filename="package://hsrb_description/meshes/arm_v0/arm_roll_light.dae" />
                 </geometry>
             </visual>
             <collision>
                 <geometry>
-                    <mesh filename="package://hsrb_meshes/meshes/arm_v0/arm_roll.stl" />
+                    <mesh filename="package://hsrb_description/meshes/arm_v0/arm_roll.stl" />
                 </geometry>
             </collision>

File: urdf/arm_v1/arm.urdf.xacro (robot description, xacro)
@@ -46,10 +46,10 @@
             <visual>
                 <geometry>
-                    <mesh filename="package://hsrb_meshes/meshes/arm_v1/shoulder.dae" />
+                    <mesh filename="package://hsrb_description/meshes/arm_v1/shoulder.dae" />
                 </geometry>
             </visual>
             <collision>
                 <geometry>
-                    <mesh filename="package://hsrb_meshes/meshes/arm_v1/shoulder.stl" />
+                    <mesh filename="package://hsrb_description/meshes/arm_v1/shoulder.stl" />
                 </geometry>
             </collision>
@@ -72,10 +72,10 @@
             <visual>
                 <geometry>
-                    <mesh filename="package://hsrb_meshes/meshes/arm_v1/arm_flex.dae" />
+                    <mesh filename="package://hsrb_description/meshes/arm_v1/arm_flex.dae" />
                 </geometry>
             </visual>
             <collision>
                 <geometry>
-                    <mesh filename="package://hsrb_meshes/meshes/arm_v1/arm_flex.stl" />
+                    <mesh filename="package://hsrb_description/meshes/arm_v1/arm_flex.stl" />
                 </geometry>
             </collision>
@@ -98,10 +98,10 @@
             <visual>
                 <geometry>
-                    <mesh filename="package://hsrb_meshes/meshes/arm_v1/arm_roll.dae" />
+                    <mesh filename="package://hsrb_description/meshes/arm_v1/arm_roll.dae" />
                 </geometry>
             </visual>
             <collision>
                 <geometry>
-                    <mesh filename="package://hsrb_meshes/meshes/arm_v1/arm_roll.stl" />
+                    <mesh filename="package://hsrb_description/meshes/arm_v1/arm_roll.stl" />
                 </geometry>
             </collision>

File: urdf/base_v2/base.urdf.xacro (robot description, xacro)
@@ -145,10 +145,10 @@
             <visual>
                 <geometry>
-                    <mesh filename="package://hsrb_meshes/meshes/base_v2/bumper.dae" />
-                </geometry>
-            </visual>
-            <collision>
-                <geometry>
-                    <mesh filename="package://hsrb_meshes/meshes/base_v2/bumper.stl" />
+                    <mesh filename="package://hsrb_description/meshes/base_v2/bumper.dae" />
+                </geometry>
+            </visual>
+            <collision>
+                <geometry>
+                    <mesh filename="package://hsrb_description/meshes/base_v2/bumper.stl" />
                 </geometry>
             </collision>
@@ -172,20 +172,20 @@
             <visual>
                 <geometry>
-                    <mesh filename="package://hsrb_meshes/meshes/base_v2/base_light.dae" />
-                </geometry>
-            </visual>
-            <visual>
-                <geometry>
-                    <mesh filename="package://hsrb_meshes/meshes/base_v2/body_light.dae" />
-                </geometry>
-            </visual>
-            <visual>
-                <geometry>
-                    <mesh filename="package://hsrb_meshes/meshes/base_v2/torso_base.dae" />
-                </geometry>
-            </visual>
-            <collision>
-                <geometry>
-                    <mesh filename="package://hsrb_meshes/meshes/base_v2/base.stl" />
+                    <mesh filename="package://hsrb_description/meshes/base_v2/base_light.dae" />
+                </geometry>
+            </visual>
+            <visual>
+                <geometry>
+                    <mesh filename="package://hsrb_description/meshes/base_v2/body_light.dae" />
+                </geometry>
+            </visual>
+            <visual>
+                <geometry>
+                    <mesh filename="package://hsrb_description/meshes/base_v2/torso_base.dae" />
+                </geometry>
+            </visual>
+            <collision>
+                <geometry>
+                    <mesh filename="package://hsrb_description/meshes/base_v2/base.stl" />
                 </geometry>
             </collision>

File: urdf/base_v3/base.urdf.xacro (robot description, xacro)
@@ -145,10 +145,10 @@
             <visual>
                 <geometry>
-                    <mesh filename="package://hsrb_meshes/meshes/base_v3/bumper.dae" />
-                </geometry>
-            </visual>
-            <collision>
-                <geometry>
-                    <mesh filename="package://hsrb_meshes/meshes/base_v3/bumper.stl" />
+                    <mesh filename="package://hsrb_description/meshes/base_v3/bumper.dae" />
+                </geometry>
+            </visual>
+            <collision>
+                <geometry>
+                    <mesh filename="package://hsrb_description/meshes/base_v3/bumper.stl" />
                 </geometry>
             </collision>
@@ -172,20 +172,20 @@
             <visual>
                 <geometry>
-                    <mesh filename="package://hsrb_meshes/meshes/base_v3/base_light.dae" />
-                </geometry>
-            </visual>
-            <visual>
-                <geometry>
-                    <mesh filename="package://hsrb_meshes/meshes/base_v3/body_light.dae" />
-                </geometry>
-            </visual>
-            <visual>
-                <geometry>
-                    <mesh filename="package://hsrb_meshes/meshes/base_v3/torso_base.dae" />
-                </geometry>
-            </visual>
-            <collision>
-                <geometry>
-                    <mesh filename="package://hsrb_meshes/meshes/base_v3/base.stl" />
+                    <mesh filename="package://hsrb_description/meshes/base_v3/base_light.dae" />
+                </geometry>
+            </visual>
+            <visual>
+                <geometry>
+                    <mesh filename="package://hsrb_description/meshes/base_v3/body_light.dae" />
+                </geometry>
+            </visual>
+            <visual>
+                <geometry>
+                    <mesh filename="package://hsrb_description/meshes/base_v3/torso_base.dae" />
+                </geometry>
+            </visual>
+            <collision>
+                <geometry>
+                    <mesh filename="package://hsrb_description/meshes/base_v3/base.stl" />
                 </geometry>
             </collision>

File: urdf/hand_v0/hand.urdf.xacro (robot description, xacro)
@@ -42,10 +42,10 @@
             <visual>
                 <geometry>
-                    <mesh filename="package://hsrb_meshes/meshes/hand_v0/palm_light.dae" />
-                </geometry>
-            </visual>
-            <collision>
-                <geometry>
-                    <mesh filename="package://hsrb_meshes/meshes/hand_v0/palm.stl" />
+                    <mesh filename="package://hsrb_description/meshes/hand_v0/palm_light.dae" />
+                </geometry>
+            </visual>
+            <collision>
+                <geometry>
+                    <mesh filename="package://hsrb_description/meshes/hand_v0/palm.stl" />
                 </geometry>
             </collision>
@@ -148,10 +148,10 @@
             <visual>
                 <geometry>
-                    <mesh filename="package://hsrb_meshes/meshes/hand_v0/l_proximal.dae" />
-                </geometry>
-            </visual>
-            <collision>
-                <geometry>
-                    <mesh filename="package://hsrb_meshes/meshes/hand_v0/l_proximal.stl" />
+                    <mesh filename="package://hsrb_description/meshes/hand_v0/l_proximal.dae" />
+                </geometry>
+            </visual>
+            <collision>
+                <geometry>
+                    <mesh filename="package://hsrb_description/meshes/hand_v0/l_proximal.stl" />
                 </geometry>
             </collision>
@@ -171,10 +171,10 @@
             <visual>
                 <geometry>
-                    <mesh filename="package://hsrb_meshes/meshes/hand_v0/l_distal.dae" />
-                </geometry>
-            </visual>
-            <collision>
-                <geometry>
-                    <mesh filename="package://hsrb_meshes/meshes/hand_v0/l_distal.stl" />
+                    <mesh filename="package://hsrb_description/meshes/hand_v0/l_distal.dae" />
+                </geometry>
+            </visual>
+            <collision>
+                <geometry>
+                    <mesh filename="package://hsrb_description/meshes/hand_v0/l_distal.stl" />
                 </geometry>
             </collision>
@@ -225,10 +225,10 @@
             <visual>
                 <geometry>
-                    <mesh filename="package://hsrb_meshes/meshes/hand_v0/r_proximal.dae" />
-                </geometry>
-            </visual>
-            <collision>
-                <geometry>
-                    <mesh filename="package://hsrb_meshes/meshes/hand_v0/r_proximal.stl" />
+                    <mesh filename="package://hsrb_description/meshes/hand_v0/r_proximal.dae" />
+                </geometry>
+            </visual>
+            <collision>
+                <geometry>
+                    <mesh filename="package://hsrb_description/meshes/hand_v0/r_proximal.stl" />
                 </geometry>
             </collision>
@@ -248,10 +248,10 @@
             <visual>
                 <geometry>
-                    <mesh filename="package://hsrb_meshes/meshes/hand_v0/r_distal.dae" />
-                </geometry>
-            </visual>
-            <collision>
-                <geometry>
-                    <mesh filename="package://hsrb_meshes/meshes/hand_v0/r_distal.stl" />
+                    <mesh filename="package://hsrb_description/meshes/hand_v0/r_distal.dae" />
+                </geometry>
+            </visual>
+            <collision>
+                <geometry>
+                    <mesh filename="package://hsrb_description/meshes/hand_v0/r_distal.stl" />
                 </geometry>
             </collision>

File: urdf/hand_v1/hand.urdf.xacro (robot description, xacro)
@@ -67,10 +67,10 @@
             <visual>
                 <geometry>
-                    <mesh filename="package://hsrb_meshes/meshes/hand_v1/palm.dae" />
-                </geometry>
-            </visual>
-            <collision>
-                <geometry>
-                    <mesh filename="package://hsrb_meshes/meshes/hand_v1/palm.stl" />
+                    <mesh filename="package://hsrb_description/meshes/hand_v1/palm.dae" />
+                </geometry>
+            </visual>
+            <collision>
+                <geometry>
+                    <mesh filename="package://hsrb_description/meshes/hand_v1/palm.stl" />
                 </geometry>
             </collision>
@@ -173,10 +173,10 @@
             <visual>
                 <geometry>
-                    <mesh filename="package://hsrb_meshes/meshes/hand_v1/l_proximal.dae" />
-                </geometry>
-            </visual>
-            <collision>
-                <geometry>
-                    <mesh filename="package://hsrb_meshes/meshes/hand_v1/l_proximal.stl" />
+                    <mesh filename="package://hsrb_description/meshes/hand_v1/l_proximal.dae" />
+                </geometry>
+            </visual>
+            <collision>
+                <geometry>
+                    <mesh filename="package://hsrb_description/meshes/hand_v1/l_proximal.stl" />
                 </geometry>
             </collision>
@@ -196,10 +196,10 @@
             <visual>
                 <geometry>
-                    <mesh filename="package://hsrb_meshes/meshes/hand_v1/l_distal.dae" />
-                </geometry>
-            </visual>
-            <collision>
-                <geometry>
-                    <mesh filename="package://hsrb_meshes/meshes/hand_v1/l_distal.stl" />
+                    <mesh filename="package://hsrb_description/meshes/hand_v1/l_distal.dae" />
+                </geometry>
+            </visual>
+            <collision>
+                <geometry>
+                    <mesh filename="package://hsrb_description/meshes/hand_v1/l_distal.stl" />
                 </geometry>
             </collision>
@@ -250,10 +250,10 @@
             <visual>
                 <geometry>
-                    <mesh filename="package://hsrb_meshes/meshes/hand_v1/r_proximal.dae" />
-                </geometry>
-            </visual>
-            <collision>
-                <geometry>
-                    <mesh filename="package://hsrb_meshes/meshes/hand_v1/r_proximal.stl" />
+                    <mesh filename="package://hsrb_description/meshes/hand_v1/r_proximal.dae" />
+                </geometry>
+            </visual>
+            <collision>
+                <geometry>
+                    <mesh filename="package://hsrb_description/meshes/hand_v1/r_proximal.stl" />
                 </geometry>
             </collision>
@@ -273,10 +273,10 @@
             <visual>
                 <geometry>
-                    <mesh filename="package://hsrb_meshes/meshes/hand_v1/r_distal.dae" />
-                </geometry>
-            </visual>
-            <collision>
-                <geometry>
-                    <mesh filename="package://hsrb_meshes/meshes/hand_v1/r_distal.stl" />
+                    <mesh filename="package://hsrb_description/meshes/hand_v1/r_distal.dae" />
+                </geometry>
+            </visual>
+            <collision>
+                <geometry>
+                    <mesh filename="package://hsrb_description/meshes/hand_v1/r_distal.stl" />
                 </geometry>
             </collision>

File: urdf/head_v2/head.urdf.xacro (robot description, xacro)
@@ -49,10 +49,10 @@
             <visual>
                 <geometry>
-                    <mesh filename="package://hsrb_meshes/meshes/head_v1/head_pan.dae" />
+                    <mesh filename="package://hsrb_description/meshes/head_v1/head_pan.dae" />
                 </geometry>
             </visual>
             <collision>
                 <geometry>
-                    <mesh filename="package://hsrb_meshes/meshes/head_v1/head_pan.stl" />
+                    <mesh filename="package://hsrb_description/meshes/head_v1/head_pan.stl" />
                 </geometry>
             </collision>
@@ -75,25 +75,25 @@
             <visual>
                 <geometry>
-                    <mesh filename="package://hsrb_meshes/meshes/head_v1/head_upper.dae" />
+                    <mesh filename="package://hsrb_description/meshes/head_v1/head_upper.dae" />
                 </geometry>
             </visual>
             <visual>
                 <geometry>
-                    <mesh filename="package://hsrb_meshes/meshes/head_v1/head_tilt.dae" />
+                    <mesh filename="package://hsrb_description/meshes/head_v1/head_tilt.dae" />
                 </geometry>
             </visual>
             <visual>
                 <geometry>
-                    <mesh filename="package://hsrb_meshes/meshes/head_v1/tablet_base.dae" />
+                    <mesh filename="package://hsrb_description/meshes/head_v1/tablet_base.dae" />
                 </geometry>
             </visual>
             <collision>
                 <geometry>
-                    <mesh filename="package://hsrb_meshes/meshes/head_v1/head.stl" />
+                    <mesh filename="package://hsrb_description/meshes/head_v1/head.stl" />
                 </geometry>
             </collision>
             <collision>
                 <geometry>
-                    <mesh filename="package://hsrb_meshes/meshes/head_v1/tablet.stl" />
+                    <mesh filename="package://hsrb_description/meshes/head_v1/tablet.stl" />
                 </geometry>
             </collision>

File: urdf/head_v3/head.urdf.xacro (robot description, xacro)
@@ -49,10 +49,10 @@
             <visual>
                 <geometry>
-                    <mesh filename="package://hsrb_meshes/meshes/head_v3/head_pan.dae" />
+                    <mesh filename="package://hsrb_description/meshes/head_v3/head_pan.dae" />
                 </geometry>
             </visual>
             <collision>
                 <geometry>
-                    <mesh filename="package://hsrb_meshes/meshes/head_v3/head_pan.stl" />
+                    <mesh filename="package://hsrb_description/meshes/head_v3/head_pan.stl" />
                 </geometry>
             </collision>
@@ -75,10 +75,10 @@
             <visual>
                 <geometry>
-                    <mesh filename="package://hsrb_meshes/meshes/head_v3/head.dae" />
+                    <mesh filename="package://hsrb_description/meshes/head_v3/head.dae" />
                 </geometry>
             </visual>
             <collision>
                 <geometry>
-                    <mesh filename="package://hsrb_meshes/meshes/head_v3/head.stl" />
+                    <mesh filename="package://hsrb_description/meshes/head_v3/head.stl" />
                 </geometry>
             </collision>

File: urdf/ros2_control.hsrb4s.robot.xacro (robot description, xacro)
@@ -26,8 +26,8 @@
 -->
 <robot xmlns:xacro="http://www.ros.org/wiki/xacro">
-  <xacro:macro name="ros2_contorl_robot">
+  <xacro:macro name="ros2_control_robot">
     <ros2_control name="hsrb" type="system">
       <hardware>
-        <plugin>hsrb_robot_hardware/HsrbHW</plugin>
+        <plugin>hsrb_description/HsrbHW</plugin>
       </hardware>
       <xacro:macro name="hsrb_joint" params="name min_angle max_angle motor_id reduction drive_mode velocity_limit gear_ratio torque_constant control_type:=ActiveJoint">

File: urdf/ros2_control.rviz.xacro (robot description, xacro)
@@ -26,8 +26,8 @@
 -->
 <robot xmlns:xacro="http://www.ros.org/wiki/xacro">
-  <xacro:macro name="ros2_contorl_rviz">
+  <xacro:macro name="ros2_control_rviz">
     <ros2_control name="GenericSystem" type="system">
       <hardware>
-        <plugin>fake_components/GenericSystem</plugin>
+        <plugin>mock_components/GenericSystem</plugin>
         <param name="fake_sensor_commands">False</param>
         <param name="state_following_offset">0.0</param>

File: urdf/sensors/asus_xtion.urdf.xacro (robot description, xacro)
@@ -12,5 +12,5 @@
                 <origin xyz="0 0 0" rpy="0.0 0.0 0.0"/>
                 <geometry>
-                    <mesh filename="package://hsrb_meshes/meshes/sensors/xtion.dae" />
+                    <mesh filename="package://hsrb_description/meshes/sensors/xtion.dae" />
                 </geometry>
             </visual>
@@ -18,5 +18,5 @@
                 <origin xyz="0 0 0" rpy="0.0 0.0 0.0"/>
                 <geometry>
-                    <mesh filename="package://hsrb_meshes/meshes/sensors/xtion.stl" />
+                    <mesh filename="package://hsrb_description/meshes/sensors/xtion.stl" />
                 </geometry>
             </collision>

File: urdf/sensors/hokuyo_laser.urdf.xacro (robot description, xacro)
@@ -12,10 +12,10 @@
             <visual>
                 <geometry>
-                    <mesh filename="package://hsrb_meshes/meshes/sensors/laser.dae" />
+                    <mesh filename="package://hsrb_description/meshes/sensors/laser.dae" />
                 </geometry>
             </visual>
             <collision>
                 <geometry>
-                    <mesh filename="package://hsrb_meshes/meshes/sensors/laser.stl" />
+                    <mesh filename="package://hsrb_description/meshes/sensors/laser.stl" />
                 </geometry>
             </collision>

File: urdf/sensors/intel_d435.urdf.xacro (robot description, xacro)
@@ -13,5 +13,5 @@
                 <origin xyz="0 0 0" rpy="0.0 0.0 0.0"/>
                 <geometry>
-                    <mesh filename="package://hsrb_meshes/meshes/sensors/xtion.dae" />
+                    <mesh filename="package://hsrb_description/meshes/sensors/xtion.dae" />
                 </geometry>
             </visual>
@@ -19,5 +19,5 @@
                 <origin xyz="0 0 0" rpy="0.0 0.0 0.0"/>
                 <geometry>
-                    <mesh filename="package://hsrb_meshes/meshes/sensors/xtion.stl" />
+                    <mesh filename="package://hsrb_description/meshes/sensors/xtion.stl" />
                 </geometry>
             </collision>
