Commit message: fixed description

File: urdf/sensors/pointgrey_chameleon.urdf.xacro (robot description, xacro)
@@ -12,5 +12,5 @@
                 <origin xyz="0 0 0" rpy="0.0 0.0 0.0"/>
                 <geometry>
-                    <mesh filename="package://hsrb_meshes/meshes/sensors/head_camera.dae" />
+                    <mesh filename="package://hsrb_description/meshes/sensors/head_camera.dae" />
                 </geometry>
             </visual>

File: urdf/torso_v0/torso.urdf.xacro (robot description, xacro)
@@ -48,10 +48,10 @@
             <visual>
                 <geometry>
-                    <mesh filename="package://hsrb_meshes/meshes/torso_v0/torso_light.dae" />
+                    <mesh filename="package://hsrb_description/meshes/torso_v0/torso_light.dae" />
                 </geometry>
             </visual>
             <collision>
                 <geometry>
-                    <mesh filename="package://hsrb_meshes/meshes/torso_v0/torso.stl" />
+                    <mesh filename="package://hsrb_description/meshes/torso_v0/torso.stl" />
                 </geometry>
             </collision>

File: urdf/torso_v1/torso.urdf.xacro (robot description, xacro)
@@ -48,10 +48,10 @@
             <visual>
                 <geometry>
-                    <mesh filename="package://hsrb_meshes/meshes/torso_v1/torso.dae" />
+                    <mesh filename="package://hsrb_description/meshes/torso_v1/torso.dae" />
                 </geometry>
             </visual>
             <collision>
                 <geometry>
-                    <mesh filename="package://hsrb_meshes/meshes/torso_v1/torso.stl" />
+                    <mesh filename="package://hsrb_description/meshes/torso_v1/torso.stl" />
                 </geometry>
             </collision>

File: urdf/wrist_v0/wrist.urdf.xacro (robot description, xacro)
@@ -47,5 +47,5 @@
             <visual>
                 <geometry>
-                    <mesh filename="package://hsrb_meshes/meshes/wrist_v0/wrist_flex.dae" />
+                    <mesh filename="package://hsrb_description/meshes/wrist_v0/wrist_flex.dae" />
                 </geometry>
                 <material name="body_sub" />
@@ -96,10 +96,10 @@
             <visual>
                 <geometry>
-                    <mesh filename="package://hsrb_meshes/meshes/wrist_v0/wrist_roll.dae" />
+                    <mesh filename="package://hsrb_description/meshes/wrist_v0/wrist_roll.dae" />
                 </geometry>
             </visual>
             <collision>
                 <geometry>
-                    <mesh filename="package://hsrb_meshes/meshes/wrist_v0/wrist_roll.stl" />
+                    <mesh filename="package://hsrb_description/meshes/wrist_v0/wrist_roll.stl" />
                 </geometry>
             </collision>

File: urdf/wrist_v1/wrist.urdf.xacro (robot description, xacro)
@@ -47,5 +47,5 @@
             <visual>
                 <geometry>
-                    <mesh filename="package://hsrb_meshes/meshes/wrist_v1/wrist_flex.dae" />
+                    <mesh filename="package://hsrb_description/meshes/wrist_v1/wrist_flex.dae" />
                 </geometry>
                 <material name="body_sub" />
@@ -96,10 +96,10 @@
             <visual>
                 <geometry>
-                    <mesh filename="package://hsrb_meshes/meshes/wrist_v1/wrist_roll.dae" />
+                    <mesh filename="package://hsrb_description/meshes/wrist_v1/wrist_roll.dae" />
                 </geometry>
             </visual>
             <collision>
                 <geometry>
-                    <mesh filename="package://hsrb_meshes/meshes/wrist_v1/wrist_roll.stl" />
+                    <mesh filename="package://hsrb_description/meshes/wrist_v1/wrist_roll.stl" />
                 </geometry>
             </collision>
